Commit message: working gazebo

File: src/urdf/two_wheel_robot.urdf (robot description, URDF)
Before this commit: robot two_wheel_robot, 3 links, 2 joints
Joints:
- joint left_joint: axis 0 -1 0 -> 0 1 0
- joint right_joint: axis 0 -1 0 -> 0 1 0

Commit message: slam

File: src/urdf/two_wheel_robot.urdf (robot description, URDF)
Before this commit: robot two_wheel_robot, 3 links, 2 joints
Links:
- added link lidar_link; collision cylinder length=0.02 radius=0.0381; visual cylinder length=0.02 radius=0.0381
Joints:
- added joint lidar_joint: type fixed, parent base_link, child lidar_link, origin xyz=0.0254 0 0.066675 rpy=0 0 0
